File: HandSTaMp.kicad_sch (KiCad schematic)
At the start: 19 parts, among them J1 USB_C_Receptacle_USB2.0_16P, J2 SDI, J3 Pins, J4 ⏚, SW1 Row 0, Col+0, SW2 Row 0, Col+1, U2 PRTR5V0U2X, U4 CH32X035G8U6

Commit message: Switch Row to PA3
This requires more trace crossings, but means that there isn’t a crossing under the MCU’s USB pads.
Parts:
- J3: PIN10 A2 -> A1; PIN11 A3 -> A2; PIN5 C15 -> C14; PIN6 C0 -> C15; PIN8 A0 -> C0; PIN9 A1 -> A0
Connections:
- net Col0: now also U4.21 (PB10); no longer U4.22 (PB11)
- net PA0: now also J3.9 (${PIN9}); no longer J3.8 (${PIN8})
- net PA1: now also J3.10 (${PIN10}); no longer J3.9 (${PIN9})
- net PA2: now also J3.11 (${PIN11}); no longer J3.10 (${PIN10})
- net PC0: now also J3.8 (${PIN8}); no longer J3.6 (${PIN6})
- net PC15: now also J3.6 (${PIN6}); no longer J3.5 (${PIN5})
- net Row0: now also U4.8 (PA3); no longer U4.21 (PB10)
- net PC14: now reaches U4.28 (PC14/CC1)
- net PC14: now also J3.5 (${PIN5})
- removed net PA3: J3.11 (${PIN11}), U4.8 (PA3)
Changed lines of the file:
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@@
 	)
 	(no_connect
-		(at 185.42 55.88)
+		(at 154.94 93.98)
 	)
 	(wire
@@
 		)
 	)
+	(global_label "PC14"
+		(shape input)
+		(at 203.2 137.16 180)
+		(fields_autoplaced yes)
+		(effects
+			(font
+				(size 1.27 1.27)
+			)
+			(justify right)
+		)
+		(property "Intersheetrefs" "${INTERSHEET_REFS}"
+			(at 196.6368 137.16 0)
+			(hide yes)
+			(show_name no)
+			(do_not_autoplace no)
+			(effects
+				(font
+					(size 1.27 1.27)
+				)
+				(justify right)
+			)
+		)
+	)
 	(global_label "Col0"
 		(shape input)
@@
 	(global_label "PA1"
 		(shape input)
-		(at 214.63 149.86 270)
+		(at 217.17 149.86 270)
 		(fields_autoplaced yes)
 		(effects
@@
 		)
 		(property "Intersheetrefs" "${INTERSHEET_REFS}"
-			(at 214.63 155.2767 90)
+			(at 217.17 155.2767 90)
 			(hide yes)
 			(show_name no)
@@
 		)
 	)
-	(global_label "PA4"
+	(global_label "Row0"
 		(shape input)
-		(at 154.94 55.88 180)
+		(at 154.94 53.34 180)
 		(fields_autoplaced yes)
 		(effects
@@
 		)
 		(property "Intersheetrefs" "${INTERSHEET_REFS}"
-			(at 149.2739 55.88 0)
+			(at 147.7664 53.34 0)
 			(hide yes)
 			(show_name no)
@@
 		)
 	)
-	(global_label "PC15"
+	(global_label "PC14"
 		(shape input)
-		(at 203.2 137.16 180)
+		(at 185.42 55.88 0)
+		(fields_autoplaced yes)
+		(effects
+			(font
+				(size 1.27 1.27)
+			)
+			(justify left)
+		)
+		(property "Intersheetrefs" "${INTERSHEET_REFS}"
+			(at 191.9832 55.88 0)
+			(hide yes)
+			(show_name no)
+			(do_not_autoplace no)
+			(effects
+				(font
+					(size 1.27 1.27)
+				)
+				(justify left)
+			)
+		)
+	)
+	(global_label "PA4"
+		(shape input)
+		(at 154.94 55.88 180)
 		(fields_autoplaced yes)
 		(effects
@@
 		)
 		(property "Intersheetrefs" "${INTERSHEET_REFS}"
-			(at 196.6902 137.16 0)
+			(at 149.2739 55.88 0)
 			(hide yes)
 			(show_name no)
@@
 		)
 	)
-	(global_label "PC0"
+	(global_label "PC15"
 		(shape input)
 		(at 203.2 139.7 180)
@@
 		)
 		(property "Intersheetrefs" "${INTERSHEET_REFS}"
-			(at 197.3949 139.7 0)
+			(at 196.6902 139.7 0)
 			(hide yes)
 			(show_name no)
@@
 		)
 	)
-	(global_label "PA3"
+	(global_label "PC0"
 		(shape input)
-		(at 154.94 53.34 180)
+		(at 203.2 144.78 180)
 		(fields_autoplaced yes)
 		(effects
@@
 		)
 		(property "Intersheetrefs" "${INTERSHEET_REFS}"
-			(at 149.3099 53.34 0)
+			(at 197.3949 144.78 0)
 			(hide yes)
 			(show_name no)
@@
 	(global_label "PA0"
 		(shape input)
-		(at 203.2 144.78 180)
+		(at 214.63 149.86 270)
 		(fields_autoplaced yes)
 		(effects
@@
 		)
 		(property "Intersheetrefs" "${INTERSHEET_REFS}"
-			(at 197.457 144.78 0)
+			(at 214.63 155.603 90)
 			(hide yes)
 			(show_name no)
@@
 		)
 	)
-	(global_label "Row0"
-		(shape input)
-		(at 154.94 91.44 180)
-		(fields_autoplaced yes)
-		(effects
-			(font
-				(size 1.27 1.27)
-			)
-			(justify right)
-		)
-		(property "Intersheetrefs" "${INTERSHEET_REFS}"
-			(at 147.7664 91.44 0)
-			(hide yes)
-			(show_name no)
-			(do_not_autoplace no)
-			(effects
-				(font
-					(size 1.27 1.27)
-				)
-				(justify right)
-			)
-		)
-	)
-	(global_label "PA2"
-		(shape input)
-		(at 217.17 149.86 270)
-		(fields_autoplaced yes)
-		(effects
-			(font
-				(size 1.27 1.27)
-			)
-			(justify right)
-		)
-		(property "Intersheetrefs" "${INTERSHEET_REFS}"
-			(at 217.17 155.4852 90)
-			(hide yes)
-			(show_name no)
-			(do_not_autoplace no)
-			(effects
-				(font
-					(size 1.27 1.27)
-				)
-				(justify right)
-			)
-		)
-	)
 	(global_label "USB+"
 		(shape bidirectional)
@@
 		)
 	)
-	(global_label "PA3"
+	(global_label "PA2"
 		(shape input)
 		(at 219.71 149.86 270)
@@
 		)
 		(property "Intersheetrefs" "${INTERSHEET_REFS}"
-			(at 219.71 155.4901 90)
+			(at 219.71 155.4852 90)
 			(hide yes)
 			(show_name no)
@@
 	(global_label "Col0"
 		(shape input)
-		(at 154.94 93.98 180)
+		(at 154.94 91.44 180)
 		(fields_autoplaced yes)
 		(effects
@@
 		)
 		(property "Intersheetrefs" "${INTERSHEET_REFS}"
-			(at 148.6064 93.98 0)
+			(at 148.6064 91.44 0)
 			(hide yes)
 			(show_name no)
@@
 			)
 		)
-		(property "PIN5" "C15"
+		(property "PIN5" "C14"
 			(at 231.14 139.7 0)
 			(hide yes)
@@
 			)
 		)
-		(property "PIN6" "C0"
+		(property "PIN6" "C15"
 			(at 231.14 139.7 0)
 			(hide yes)
@@
 			)
 		)
-		(property "PIN8" "A0"
+		(property "PIN8" "C0"
 			(at 231.14 139.7 0)
 			(hide yes)
@@
 			)
 		)
-		(property "PIN9" "A1"
+		(property "PIN9" "A0"
 			(at 231.14 139.7 0)
 			(hide yes)
@@
 			)
 		)
-		(property "PIN10" "A2"
+		(property "PIN10" "A1"
 			(at 231.14 139.7 0)
 			(hide yes)
@@
 			)
 		)
-		(property "PIN11" "A3"
+		(property "PIN11" "A2"
 			(at 231.14 139.7 0)
 			(hide yes)
